File: 258D.kicad_pcb (KiCad board)
At the start: 2 copper layers, 104 x 158 mm, 227 parts, among them J1 +15V, J101 Vary CV 1, J102 Vary CV 2, J103 V/O, J104 FM IN, J105 Shape CV, J106 SHAPE SEL 1, J107 SHAPE SEL 3, J108 SHAPE SEL 2, J109 Triangle Out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

Commit message: Update BOM, BOM pdf, notes, schematic
Parts:
- C101, C201: value 4n7 -> 2n2

Commit message: Update Q104/204 value in schematic, board, BOM, iBOM, clarify selection criteria for Q105/205 in schematic, BOM, notes.
Parts:
- Q104, Q204: value MMBF5484 -> MMBF5485
