File: 258D.sch (KiCad schematic (older format))
At the start: 31 parts, among them J1 +15V, J2 0V, J3 -15V, M1 Logo_150mil, M2 Mod_Indicator_1-10_150mil, M3 Serial_Box_150mil, U1 ADR01, U2 TL071

Commit message: Update BOM, BOM pdf, notes, schematic
Parts:
- M1: symbol Dunnington:Logo_150mil -> 258D-rescue:Logo_150mil-Dunnington
- M2: symbol Dunnington:Mod_Indicator_1-10_150mil -> 258D-rescue:Mod_Indicator_1-10_150mil-Dunnington
- M3: symbol Dunnington:Serial_Box_150mil -> 258D-rescue:Serial_Box_150mil-Dunnington
Changed lines of the file:
@@
 $EndComp
 $Comp
-L Dunnington:Mod_Indicator_1-10_150mil M2
+L 258D-rescue:Mod_Indicator_1-10_150mil-Dunnington M2
 U 1 1 5E569A04
 P 5000 9000
@@
 $EndComp
 $Comp
-L Dunnington:Serial_Box_150mil M3
+L 258D-rescue:Serial_Box_150mil-Dunnington M3
 U 1 1 5E56A955
 P 5000 9275
@@
 $EndComp
 $Comp
-L Dunnington:Logo_150mil M1
+L 258D-rescue:Logo_150mil-Dunnington M1
 U 1 1 5E5A3AC1
 P 5000 8700

Commit message: Update Q104/204 value in schematic, board, BOM, iBOM, clarify selection criteria for Q105/205 in schematic, BOM, notes.
Parts:
- U1: symbol AnalogDevices:ADR01 -> 258D-rescue:ADR01-AnalogDevices
Changed lines of the file:
@@
 	5750 7500 6000 7500
 $Comp
-L AnalogDevices:ADR01 U1
+L 258D-rescue:ADR01-AnalogDevices U1
 U 1 1 5D02CBA7
 P 2050 7225
