File: 258D_Cell.sch (KiCad schematic (older format))
At the start: 98 parts, among them J101 Vary CV 1, J102 Vary CV 2, J103 V/O, J104 FM IN, J105 Shape CV, J106 SHAPE SEL 1, J107 SHAPE SEL 3, J108 SHAPE SEL 2, J109 Triangle Out, J110 Final Out 1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

Commit message: Update BOM, BOM pdf, notes, schematic
Parts:
- C101: value 4n7 -> 2n2
Other:
- note added: "NOTES\n\nSelect R105/R205 for V/O scale other than 1.2 V/O\n\nTo match coarse frequency front panel scale R103/203 = 150k\nFor reduced range R103/203 = 180k\n\nSelect Q105/205 for VGS(off) of 1.13V for best sine shape\n\nShape select headers:\nConnect pins 1 & 2 for square\nConnect pins 2 & 3 for saw\n\nC101/C201 changed to 2n2 for improved tracking 20200629"
- note removed: "NOTES\n\nSelect R105/R205 for V/O scale other than 1.2 V/O\n\nTo match coarse frequency front panel scale R103/203 = 150k\nFor reduced range R103/203 = 180k\n\nSelect Q105/205 for VGS(off) of 1.13V for best sine shape\n\nShape select headers:\nConnect pins 1 & 2 for square\nConnect pins 2 & 3 for saw"
Changed lines of the file:
@@
 AR Path="/5D075473/5D0F6500" Ref="C201"  Part="1"
 F 0 "C101" V 7600 2225 50  0000 L CNN
-F 1 "4n7" V 7500 2325 50  0000 C CNN
+F 1 "2n2" V 7500 2325 50  0000 C CNN
 F 2 "Capacitor_SMD:C_0805_2012Metric" H 7550 2325 50  0001 C CNN
 F 3 "" H 7550 2475 50  0001 C CNN
@@
 ~~4.5Vp-p (Sine)
 Text Notes 13000 8800 0    50   ~ 0
-NOTES\n\nSelect R105/R205 for V/O scale other than 1.2 V/O\n\nTo match coarse frequency front panel scale R103/203 = 150k\nFor reduced range R103/203 = 180k\n\nSelect Q105/205 for VGS(off) of 1.13V for best sine shape\n\nShape select headers:\nConnect pins 1 & 2 for square\nConnect pins 2 & 3 for saw
+NOTES\n\nSelect R105/R205 for V/O scale other than 1.2 V/O\n\nTo match coarse frequency front panel scale R103/203 = 150k\nFor reduced range R103/203 = 180k\n\nSelect Q105/205 for VGS(off) of 1.13V for best sine shape\n\nShape select headers:\nConnect pins 1 & 2 for square\nConnect pins 2 & 3 for saw\n\nC101/C201 changed to 2n2 for improved tracking 20200629
 Wire Wire Line
 	9750 6100 9750 6200

Commit message: Update Q104/204 value in schematic, board, BOM, iBOM, clarify selection criteria for Q105/205 in schematic, BOM, notes.
Parts:
- Q101: symbol DiodesInc:DMMT3906W -> 258D-rescue:DMMT3906W-DiodesInc
- Q102: symbol DiodesInc:DMMT3904W -> 258D-rescue:DMMT3904W-DiodesInc
- Q103: symbol OnSemiconductor:MMBT3906 -> 258D-rescue:MMBT3906-OnSemiconductor
- Q104: value MMBF5484 -> MMBF5485; symbol OnSemiconductor:MMBFJ201 -> 258D-rescue:MMBFJ201-OnSemiconductor
- Q105: symbol OnSemiconductor:MMBFJ201 -> 258D-rescue:MMBFJ201-OnSemiconductor
- VR101, VR102, VR103, VR104, VR105, VR106: symbol TaiwanAlpha:POT -> 258D-rescue:POT-TaiwanAlpha
Other:
- note added: "NOTES\n\nSelect R105/R205 for V/O scale other than 1.2 V/O\n\nTo match coarse frequency front panel scale R103/203 = 150k\nFor reduced range R103/203 = 180k\n\nSelect Q105/205 for VGS(off) of 0.8V - 1.2V. Ideal value is 1.13V\nfor best sine shape\n\nShape select headers:\nConnect pins 1 & 2 for square\nConnect pins 2 & 3 for saw\n\nC101/C201 changed to 2n2 for improved tracking 20200629"
- note removed: "NOTES\n\nSelect R105/R205 for V/O scale other than 1.2 V/O\n\nTo match coarse frequency front panel scale R103/203 = 150k\nFor reduced range R103/203 = 180k\n\nSelect Q105/205 for VGS(off) of 1.13V for best sine shape\n\nShape select headers:\nConnect pins 1 & 2 for square\nConnect pins 2 & 3 for saw\n\nC101/C201 changed to 2n2 for improved tracking 20200629"
Changed lines of the file:
@@
 $EndComp
 $Comp
-L TaiwanAlpha:POT VR?
+L 258D-rescue:POT-TaiwanAlpha VR?
 U 1 1 5D0F643A
 P 8375 7400
@@
 AR Path="/5D0750F6/5D0F643A" Ref="VR106"  Part="1"
 AR Path="/5D075473/5D0F643A" Ref="VR206"  Part="1"
+AR Path="/5D0F643A" Ref="VR106"  Part="1"
 F 0 "VR106" V 8200 7400 50  0000 C CNN
 F 1 "100kB" V 8275 7400 50  0000 C CNN
@@
 $EndComp
 $Comp
-L OnSemiconductor:MMBFJ201 Q?
+L 258D-rescue:MMBFJ201-OnSemiconductor Q?
 U 1 1 5D0F6488
 P 9850 5650
@@
 AR Path="/5D0750F6/5D0F6488" Ref="Q104"  Part="1"
 AR Path="/5D075473/5D0F6488" Ref="Q204"  Part="1"
+AR Path="/5D0F6488" Ref="Q104"  Part="1"
 F 0 "Q104" V 9800 5500 50  0000 R CNN
-F 1 "MMBF5484" V 9700 5500 50  0000 R CNN
+F 1 "MMBF5485" V 9700 5500 50  0000 R CNN
 F 2 "Package_TO_SOT_SMD:SOT-23" H 10050 5575 50  0001 L CIN
 F 3 "" H 9850 5600 50  0001 L CNN
@@
 $EndComp
 $Comp
-L OnSemiconductor:MMBFJ201 Q?
+L 258D-rescue:MMBFJ201-OnSemiconductor Q?
 U 1 1 5D0F64AC
 P 10100 4700
@@
 AR Path="/5D0750F6/5D0F64AC" Ref="Q105"  Part="1"
 AR Path="/5D075473/5D0F64AC" Ref="Q205"  Part="1"
+AR Path="/5D0F64AC" Ref="Q105"  Part="1"
 F 0 "Q105" H 10275 4725 50  0000 L CNN
 F 1 "MMBFJ201" H 10275 4650 50  0000 L CNN
@@
 $EndComp
 $Comp
-L OnSemiconductor:MMBT3906 Q?
+L 258D-rescue:MMBT3906-OnSemiconductor Q?
 U 1 1 5D0F64C4
 P 8900 2100
@@
 AR Path="/5D0750F6/5D0F64C4" Ref="Q103"  Part="1"
 AR Path="/5D075473/5D0F64C4" Ref="Q203"  Part="1"
+AR Path="/5D0F64C4" Ref="Q103"  Part="1"
 F 0 "Q103" H 9100 2075 50  0000 L CNN
 F 1 "MMBT3906" H 9100 2150 50  0000 L CNN
@@
 $EndComp
 $Comp
-L DiodesInc:DMMT3904W Q?
+L 258D-rescue:DMMT3904W-DiodesInc Q?
 U 2 1 5D0F64F4
 P 8700 2950
@@
 $EndComp
 $Comp
-L DiodesInc:DMMT3904W Q?
+L 258D-rescue:DMMT3904W-DiodesInc Q?
 U 1 1 5D0F64FA
 P 8150 2950
@@
 $EndComp
 $Comp
-L TaiwanAlpha:POT VR?
+L 258D-rescue:POT-TaiwanAlpha VR?
 U 1 1 5D0F657E
 P 3050 5400
@@
 AR Path="/5D0750F6/5D0F657E" Ref="VR105"  Part="1"
 AR Path="/5D075473/5D0F657E" Ref="VR205"  Part="1"
+AR Path="/5D0F657E" Ref="VR105"  Part="1"
 F 0 "VR105" V 2875 5400 50  0000 C CNN
 F 1 "100kA" V 2950 5400 50  0000 C CNN
@@
 $EndComp
 $Comp
-L DiodesInc:DMMT3906W Q?
+L 258D-rescue:DMMT3906W-DiodesInc Q?
 U 1 1 5D0F659C
 P 5050 6150
@@
 $EndComp
 $Comp
-L DiodesInc:DMMT3906W Q?
+L 258D-rescue:DMMT3906W-DiodesInc Q?
 U 2 1 5D0F65A2
 P 4650 6150
@@
 $EndComp
 $Comp
-L TaiwanAlpha:POT VR?
+L 258D-rescue:POT-TaiwanAlpha VR?
 U 1 1 5D0F65D2
 P 2650 4300
@@
 AR Path="/5D0750F6/5D0F65D2" Ref="VR102"  Part="1"
 AR Path="/5D075473/5D0F65D2" Ref="VR202"  Part="1"
+AR Path="/5D0F65D2" Ref="VR102"  Part="1"
 F 0 "VR102" V 2475 4300 50  0000 C CNN
 F 1 "100kB" V 2550 4300 50  0000 C CNN
@@
 $EndComp
 $Comp
-L TaiwanAlpha:POT VR?
+L 258D-rescue:POT-TaiwanAlpha VR?
 U 1 1 5D0F65D8
 P 2650 3600
@@
 AR Path="/5D0750F6/5D0F65D8" Ref="VR101"  Part="1"
 AR Path="/5D075473/5D0F65D8" Ref="VR201"  Part="1"
+AR Path="/5D0F65D8" Ref="VR101"  Part="1"
 F 0 "VR101" V 2475 3600 50  0000 C CNN
 F 1 "100kB" V 2550 3600 50  0000 C CNN
@@
 $EndComp
 $Comp
-L TaiwanAlpha:POT VR?
+L 258D-rescue:POT-TaiwanAlpha VR?
 U 1 1 5D0F6608
 P 3000 2950
@@
 AR Path="/5D0750F6/5D0F6608" Ref="VR104"  Part="1"
 AR Path="/5D075473/5D0F6608" Ref="VR204"  Part="1"
+AR Path="/5D0F6608" Ref="VR104"  Part="1"
 F 0 "VR104" V 2900 2950 50  0000 C CNN
 F 1 "100kB" V 2825 2950 50  0000 C CNN
@@
 $EndComp
 $Comp
-L TaiwanAlpha:POT VR?
+L 258D-rescue:POT-TaiwanAlpha VR?
 U 1 1 5D0F660E
 P 3000 2300
@@
 AR Path="/5D0750F6/5D0F660E" Ref="VR103"  Part="1"
 AR Path="/5D075473/5D0F660E" Ref="VR203"  Part="1"
+AR Path="/5D0F660E" Ref="VR103"  Part="1"
 F 0 "VR103" V 2900 2300 50  0000 C CNN
 F 1 "100kB" V 2825 2300 50  0000 C CNN
@@
 ~~4.5Vp-p (Sine)
 Text Notes 13000 8800 0    50   ~ 0
-NOTES\n\nSelect R105/R205 for V/O scale other than 1.2 V/O\n\nTo match coarse frequency front panel scale R103/203 = 150k\nFor reduced range R103/203 = 180k\n\nSelect Q105/205 for VGS(off) of 1.13V for best sine shape\n\nShape select headers:\nConnect pins 1 & 2 for square\nConnect pins 2 & 3 for saw\n\nC101/C201 changed to 2n2 for improved tracking 20200629
+NOTES\n\nSelect R105/R205 for V/O scale other than 1.2 V/O\n\nTo match coarse frequency front panel scale R103/203 = 150k\nFor reduced range R103/203 = 180k\n\nSelect Q105/205 for VGS(off) of 0.8V - 1.2V. Ideal value is 1.13V\nfor best sine shape\n\nShape select headers:\nConnect pins 1 & 2 for square\nConnect pins 2 & 3 for saw\n\nC101/C201 changed to 2n2 for improved tracking 20200629
 Wire Wire Line
 	9750 6100 9750 6200
